File: hardware/esp32_led_controller.sch (KiCad schematic (older format))
At the start: 28 parts, among them J1 USB_B, J2 BARREL_JACK, J3 Screw_Terminal_1x03, J4 CONN_01X11, J5 CONN_01X09, Q1 Q_NPN_BEC, Q4 Q_NPN_BEC, SW1 SW_Push, U1 MCP1415, U11 AZ1117-3.3, U3 CP2102, U4 ESP32-WROOM-32

Commit message: Finished design with integrated LED matrix
Parts:
- removed J3: Screw_Terminal_1x03, TerminalBlock_TE-Connectivity:TerminalBlock_TE_282834-3_1x03_P2.54mm_Horizontal, symbol conn:Screw_Terminal_1x03
- removed J4: CONN_01X11, Connector_PinHeader_2.54mm:PinHeader_1x11_P2.54mm_Vertical, symbol conn:CONN_01X11
- added C265: 1000uF, Capacitor_SMD:CP_Elec_10x10, symbol Device:CP
- added D257: R, LED_SMD:LED_0603_1608Metric, symbol Device:LED
- added D258: G, LED_SMD:LED_0603_1608Metric, symbol Device:LED
- added D259: Y, LED_SMD:LED_0603_1608Metric, symbol Device:LED
- added H1, H2, H3, H4: MountingHole, MountingHole:MountingHole_2.2mm_M2, symbol Mechanical:MountingHole
- added J3: CONN_01X08, Connector_PinHeader_2.54mm:PinHeader_1x08_P2.54mm_Vertical, symbol conn:CONN_01X08
- added J5: CONN_01X03, Connector_PinHeader_2.54mm:PinHeader_1x03_P2.54mm_Vertical, symbol conn:CONN_01X03
- added J6: USB_C_Receptacle_USB2.0, Connector_USB:USB_C_Receptacle_HRO_TYPE-C-31-M-12, symbol Connector:USB_C_Receptacle_USB2.0
- added R10, R8, R9: 100R, Resistor_SMD:R_0402_1005Metric, symbol Device:R
- added R11, R12: 5.1kR, Resistor_SMD:R_0402_1005Metric, symbol Device:R
- added R3: 470R, Resistor_SMD:R_0402_1005Metric, symbol Device:R
- added TP3: TestPoint, TestPoint:TestPoint_Loop_D3.50mm_Drill1.4mm_Beaded, symbol Connector:TestPoint
- J1: symbol Connector:USB_B -> esp32_led_controller-rescue:USB_B-Connector
- J4: renamed from J2; footprint Connector_BarrelJack:BarrelJack_Wuerth_6941xx301002 -> dc_jack:DC-005C-25A; LCSC (none) -> C223903
- renumbered C3 to C2, C4 to C3, C10 to C4, C9 to C5, J5 to J2, Q4 to Q2, R28 to R1, R25 to R2, R27 to R4, R18 to R5, R16 to R6, R17 to R7, TP2 to TP1, TP1 to TP2, U3 to U2, U4 to U3, U11 to U4
Connections:
- net IO27 is gone; now on net DOUT: U3.12 (IO27)
- net +3V3: now also J3.1 (P1)
- net +5V: now also C265.1, J3.2 (P2), J5.1 (P1)
- net DOUT: no longer U3.37 (IO23)
- net GND: now also C265.2, J3.8 (P8), J5.3 (P3), J6.A1 (GND), J6.A12 (GND), J6.B1 (GND), J6.B12 (GND), J6.S1 (SHIELD), R10.1, R11.1, R12.1, R8.1, R9.1
- net IO25: now also D258.2 (A)
- net IO26: now also D257.2 (A)
- net IO32: now also J3.7 (P7)
- net IO33: now also D259.2 (A)
- net IO34: now also J3.5 (P5)
- net IO35: now also J3.6 (P6)
- net IO36: now also J3.3 (P3)
- net IO39: now also J3.4 (P4)
- net Vbus: now reaches J1.1 (VBUS), R4.2, U2.8 (VBUS)
- net Vbus: now also J6.A4 (VBUS), J6.A9 (VBUS), J6.B4 (VBUS), J6.B9 (VBUS)
- net Dm: now reaches J1.2 (D-), U2.5 (D-)
- net Dm: now also J6.A7 (D-), J6.B7 (D-)
- net Dp: now reaches J1.3 (D+), U2.4 (D+)
- net Dp: now also J6.A6 (D+), J6.B6 (D+)
- net at U1.5 (~OUT): now also R3.2
- new net: D257.1 (K), R8.2
- new net: D258.1 (K), R9.2
- new net: D259.1 (K), R10.2
- new net: J6.A5 (CC1), R11.2
- new net: J6.B5 (CC2), R12.2
- new net LED_SIG: R3.1, TP3.1
- new net row7/Dout: J5.2 (P2)
Other:
- note added: "LEDs"
- note added: "Level Shifter"
- note added: "Mechanical"
- note added: "These pull-down resistors tell the host we are\nan UFP. Only one is used for a given connection,\nbut we need both for reversibility."
- note added: "USB Connectors"
- note added: "USB-Serial"
- note removed: "Barrel Jack:\n2.5mm ID: 694108301002 \n2.1mm ID: 694106301002"
- note removed: "LED Connector"
- note removed: "TE 282834-3"
- note removed: "USB"
- moved on the sheet: C2, C3, C6, C7, C8, J1, J4, Q1, Q2, R1, R4, R5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
