File: hardware/esp32_led_controller/esp32_led_controller.sch (KiCad schematic (older format))
At the start: 44 parts, among them J1 USB_B, J2 CONN_01X09, J3 CONN_01X08, J4 BARREL_JACK, J5 CONN_01X03, J6 USB_C_Receptacle_USB2.0, Q1 Q_NPN_BEC, Q2 Q_NPN_BEC, SW1 SW_Push, U1 MCP1415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

Commit message: Improved silkscreen and added test points
Parts:
- added R13: 10kR, Resistor_SMD:R_0402_1005Metric, symbol Device:R
- added TP? (x2): TestPoint, TestPoint:TestPoint_Loop_D3.50mm_Drill1.4mm_Beaded, symbol Connector:TestPoint
Connections:
- net +3V3: now also R13.2
- net DOUT: now also R13.1
- net EN: now also TP?.1
- net IO0: now also TP?.1
Other:
- moved on the sheet: D257, D258, D259, R10, R8, R9
Changed lines of the file:
@@
 IO0
 Wire Wire Line
-	2300 9300 2300 9450
+	2300 9300 2300 9350
 Wire Notes Line
 	850  9500 850  8000
@@
 	2300 8200 2300 8250
 Wire Wire Line
-	2300 8250 3000 8250
+	2300 8250 2600 8250
 Wire Wire Line
 	3000 8250 3000 8700
@@
 	1    0    0    -1
 $EndComp
-Text Label 6700 3700 0    60   ~ 0
+Text Label 7400 3700 0    60   ~ 0
 DOUT
 Text Label 8450 2050 2    60   ~ 0
@@
 Text Label 8450 4000 2    50   ~ 0
 IO32
-Text Label 11100 3600 2    50   ~ 0
+Text Label 11350 3350 2    50   ~ 0
 IO33
 Text Label 6700 3500 0    50   ~ 0
@@
 IO26
 Wire Wire Line
-	6550 3700 6700 3700
-Wire Wire Line
 	6700 3600 6550 3600
 Wire Wire Line
 	6550 3500 6700 3500
-Text Label 10750 3600 2    50   ~ 0
+Text Label 11000 3350 2    50   ~ 0
 IO25
-Text Label 10350 3600 2    50   ~ 0
+Text Label 10600 3350 2    50   ~ 0
 IO26
 $Comp
@@
 L Device:LED D257
 U 1 1 606D03EF
-P 10400 3800
-F 0 "D257" V 10439 3682 50  0000 R CNN
-F 1 "R" V 10348 3682 50  0000 R CNN
-F 2 "LED_SMD:LED_0603_1608Metric" H 10400 3800 50  0001 C CNN
-F 3 "~" H 10400 3800 50  0001 C CNN
-F 4 "C72044" V 10400 3800 50  0001 C CNN "LCSC"
-	1    10400 3800
+P 10650 3550
+F 0 "D257" V 10689 3432 50  0000 R CNN
+F 1 "R" V 10598 3432 50  0000 R CNN
+F 2 "LED_SMD:LED_0603_1608Metric" H 10650 3550 50  0001 C CNN
+F 3 "~" H 10650 3550 50  0001 C CNN
+F 4 "C72044" V 10650 3550 50  0001 C CNN "LCSC"
+	1    10650 3550
 	0    -1   -1   0
 $EndComp
@@
 L Device:LED D258
 U 1 1 606D10AE
-P 10800 3800
-F 0 "D258" V 10839 3682 50  0000 R CNN
-F 1 "G" V 10748 3682 50  0000 R CNN
-F 2 "LED_SMD:LED_0603_1608Metric" H 10800 3800 50  0001 C CNN
-F 3 "~" H 10800 3800 50  0001 C CNN
-F 4 "C72043" V 10800 3800 50  0001 C CNN "LCSC"
-	1    10800 3800
+P 11050 3550
+F 0 "D258" V 11089 3432 50  0000 R CNN
+F 1 "G" V 10998 3432 50  0000 R CNN
+F 2 "LED_SMD:LED_0603_1608Metric" H 11050 3550 50  0001 C CNN
+F 3 "~" H 11050 3550 50  0001 C CNN
+F 4 "C72043" V 11050 3550 50  0001 C CNN "LCSC"
+	1    11050 3550
 	0    -1   -1   0
 $EndComp
@@
 L Device:LED D259
 U 1 1 606D15D2
-P 11150 3800
-F 0 "D259" V 11189 3682 50  0000 R CNN
-F 1 "Y" V 11098 3682 50  0000 R CNN
-F 2 "LED_SMD:LED_0603_1608Metric" H 11150 3800 50  0001 C CNN
-F 3 "~" H 11150 3800 50  0001 C CNN
-F 4 "C72038" V 11150 3800 50  0001 C CNN "LCSC"
-	1    11150 3800
+P 11400 3550
+F 0 "D259" V 11439 3432 50  0000 R CNN
+F 1 "Y" V 11348 3432 50  0000 R CNN
+F 2 "LED_SMD:LED_0603_1608Metric" H 11400 3550 50  0001 C CNN
+F 3 "~" H 11400 3550 50  0001 C CNN
+F 4 "C72038" V 11400 3550 50  0001 C CNN "LCSC"
+	1    11400 3550
 	0    -1   -1   0
 $EndComp
 Wire Wire Line
-	10350 3600 10400 3600
-Wire Wire Line
-	10400 3600 10400 3650
-Wire Wire Line
-	10750 3600 10800 3600
-Wire Wire Line
-	10800 3600 10800 3650
-Wire Wire Line
-	11100 3600 11150 3600
-Wire Wire Line
-	11150 3600 11150 3650
+	10600 3350 10650 3350
+Wire Wire Line
+	10650 3350 10650 3400
+Wire Wire Line
+	11000 3350 11050 3350
+Wire Wire Line
+	11050 3350 11050 3400
+Wire Wire Line
+	11350 3350 11400 3350
+Wire Wire Line
+	11400 3350 11400 3400
 $Comp
 L Device:R R8
 U 1 1 606DE191
-P 10400 4200
-F 0 "R8" V 10193 4200 50  0000 C CNN
-F 1 "100R" V 10284 4200 50  0000 C CNN
-F 2 "Resistor_SMD:R_0402_1005Metric" V 10330 4200 50  0001 C CNN
-F 3 "~" H 10400 4200 50  0001 C CNN
-F 4 "C25076" V 10400 4200 50  0001 C CNN "LCSC"
-	1    10400 4200
+P 10650 3950
+F 0 "R8" V 10443 3950 50  0000 C CNN
+F 1 "100R" V 10534 3950 50  0000 C CNN
+F 2 "Resistor_SMD:R_0402_1005Metric" V 10580 3950 50  0001 C CNN
+F 3 "~" H 10650 3950 50  0001 C CNN
+F 4 "C25076" V 10650 3950 50  0001 C CNN "LCSC"
+	1    10650 3950
 	-1   0    0    1
 $EndComp
@@
 L Device:R R9
 U 1 1 606DE7FE
-P 10800 4200
-F 0 "R9" V 10593 4200 50  0000 C CNN
-F 1 "100R" V 10684 4200 50  0000 C CNN
-F 2 "Resistor_SMD:R_0402_1005Metric" V 10730 4200 50  0001 C CNN
-F 3 "~" H 10800 4200 50  0001 C CNN
-F 4 "C25076" V 10800 4200 50  0001 C CNN "LCSC"
-	1    10800 4200
+P 11050 3950
+F 0 "R9" V 10843 3950 50  0000 C CNN
+F 1 "100R" V 10934 3950 50  0000 C CNN
+F 2 "Resistor_SMD:R_0402_1005Metric" V 10980 3950 50  0001 C CNN
+F 3 "~" H 11050 3950 50  0001 C CNN
+F 4 "C25076" V 11050 3950 50  0001 C CNN "LCSC"
+	1    11050 3950
 	-1   0    0    1
 $EndComp
@@
 L Device:R R10
 U 1 1 606DEA2D
-P 11150 4200
-F 0 "R10" V 10943 4200 50  0000 C CNN
-F 1 "100R" V 11034 4200 50  0000 C CNN
-F 2 "Resistor_SMD:R_0402_1005Metric" V 11080 4200 50  0001 C CNN
-F 3 "~" H 11150 4200 50  0001 C CNN
-F 4 "C25076" V 11150 4200 50  0001 C CNN "LCSC"
-	1    11150 4200
+P 11400 3950
+F 0 "R10" V 11193 3950 50  0000 C CNN
+F 1 "100R" V 11284 3950 50  0000 C CNN
+F 2 "Resistor_SMD:R_0402_1005Metric" V 11330 3950 50  0001 C CNN
+F 3 "~" H 11400 3950 50  0001 C CNN
+F 4 "C25076" V 11400 3950 50  0001 C CNN "LCSC"
+	1    11400 3950
 	-1   0    0    1
 $EndComp
@@
 L power:GND #PWR?
 U 1 1 606DED03
-P 10400 4450
+P 10650 4200
 AR Path="/5F1ED570/606DED03" Ref="#PWR?"  Part="1"
 AR Path="/606DED03" Ref="#PWR01066"  Part="1"
-F 0 "#PWR01066" H 10400 4200 50  0001 C CNN
-F 1 "GND" H 10405 4277 50  0000 C CNN
-F 2 "" H 10400 4450 50  0001 C CNN
-F 3 "" H 10400 4450 50  0001 C CNN
-	1    10400 4450
+F 0 "#PWR01066" H 10650 3950 50  0001 C CNN
+F 1 "GND" H 10655 4027 50  0000 C CNN
+F 2 "" H 10650 4200 50  0001 C CNN
+F 3 "" H 10650 4200 50  0001 C CNN
+	1    10650 4200
 	1    0    0    -1
 $EndComp
@@
 L power:GND #PWR?
 U 1 1 606DF0F7
-P 10800 4450
+P 11050 4200
 AR Path="/5F1ED570/606DF0F7" Ref="#PWR?"  Part="1"
 AR Path="/606DF0F7" Ref="#PWR01067"  Part="1"
-F 0 "#PWR01067" H 10800 4200 50  0001 C CNN
-F 1 "GND" H 10805 4277 50  0000 C CNN
-F 2 "" H 10800 4450 50  0001 C CNN
-F 3 "" H 10800 4450 50  0001 C CNN
-	1    10800 4450
+F 0 "#PWR01067" H 11050 3950 50  0001 C CNN
+F 1 "GND" H 11055 4027 50  0000 C CNN
+F 2 "" H 11050 4200 50  0001 C CNN
+F 3 "" H 11050 4200 50  0001 C CNN
+	1    11050 4200
 	1    0    0    -1
 $EndComp
@@
 L power:GND #PWR?
 U 1 1 606DF332
-P 11150 4450
+P 11400 4200
 AR Path="/5F1ED570/606DF332" Ref="#PWR?"  Part="1"
 AR Path="/606DF332" Ref="#PWR01068"  Part="1"
-F 0 "#PWR01068" H 11150 4200 50  0001 C CNN
-F 1 "GND" H 11155 4277 50  0000 C CNN
-F 2 "" H 11150 4450 50  0001 C CNN
-F 3 "" H 11150 4450 50  0001 C CNN
-	1    11150 4450
-	1    0    0    -1
-$EndComp
-Wire Wire Line
-	11150 4450 11150 4350
-Wire Wire Line
-	10800 4350 10800 4450
-Wire Wire Line
-	10400 4350 10400 4450
-Wire Wire Line
-	10400 3950 10400 4050
-Wire Wire Line
-	10800 3950 10800 4050
-Wire Wire Line
-	11150 3950 11150 4050
+F 0 "#PWR01068" H 11400 3950 50  0001 C CNN
+F 1 "GND" H 11405 4027 50  0000 C CNN
+F 2 "" H 11400 4200 50  0001 C CNN
+F 3 "" H 11400 4200 50  0001 C CNN
+	1    11400 4200
+	1    0    0    -1
+$EndComp
+Wire Wire Line
+	11400 4200 11400 4100
+Wire Wire Line
+	11050 4100 11050 4200
+Wire Wire Line
+	10650 4100 10650 4200
+Wire Wire Line
+	10650 3700 10650 3800
+Wire Wire Line
+	11050 3700 11050 3800
+Wire Wire Line
+	11400 3700 11400 3800
 $Comp
 L Connector:USB_C_Receptacle_USB2.0 J6
@@
 	1    0    0    -1
 $EndComp
-Text Notes 2550 1750 0    39   ~ 0
+Text Notes 2500 1750 0    39   ~ 0
 These pull-down resistors tell the host we are\nan UFP. Only one is used for a given connection,\nbut we need both for reversibility.
 Text Label 2250 2300 0    50   ~ 0
@@
 Wire Wire Line
 	2150 2100 2150 2150
+$Comp
+L Device:R R?
+U 1 1 60242CDB
+P 7200 3550
+AR Path="/5F1ED570/60242CDB" Ref="R?"  Part="1"
+AR Path="/60242CDB" Ref="R13"  Part="1"
+F 0 "R13" H 7400 3500 50  0000 R CNN
+F 1 "10kR" H 7450 3600 50  0000 R CNN
+F 2 "Resistor_SMD:R_0402_1005Metric" V 7130 3550 50  0001 C CNN
+F 3 "~" H 7200 3550 50  0001 C CNN
+F 4 "C25744" V 7200 3550 50  0001 C CNN "LCSC"
+	1    7200 3550
+	-1   0    0    1
+$EndComp
+Wire Wire Line
+	7400 3700 7200 3700
+Wire Wire Line
+	6550 3700 7200 3700
+Connection ~ 7200 3700
+$Comp
+L power:+3V3 #PWR?
+U 1 1 60250FC6
+P 7200 3400
+AR Path="/5F1ED570/60250FC6" Ref="#PWR?"  Part="1"
+AR Path="/60250FC6" Ref="#PWR01073"  Part="1"
+F 0 "#PWR01073" H 7200 3250 50  0001 C CNN
+F 1 "+3V3" H 7215 3573 50  0000 C CNN
+F 2 "" H 7200 3400 50  0001 C CNN
+F 3 "" H 7200 3400 50  0001 C CNN
+	1    7200 3400
+	1    0    0    -1
+$EndComp
+$Comp
+L Connector:TestPoint TP?
+U 1 1 6025CD38
+P 2600 8200
+F 0 "TP?" H 2658 8318 50  0000 L CNN
+F 1 "TestPoint" H 2658 8227 50  0000 L CNN
+F 2 "TestPoint:TestPoint_Loop_D3.50mm_Drill1.4mm_Beaded" H 2800 8200 50  0001 C CNN
+F 3 "~" H 2800 8200 50  0001 C CNN
+	1    2600 8200
+	1    0    0    -1
+$EndComp
+$Comp
+L Connector:TestPoint TP?
+U 1 1 6025DADF
+P 2550 9350
+F 0 "TP?" H 2608 9468 50  0000 L CNN
+F 1 "TestPoint" H 2550 9350 50  0000 L CNN
+F 2 "TestPoint:TestPoint_Loop_D3.50mm_Drill1.4mm_Beaded" H 2750 9350 50  0001 C CNN
+F 3 "~" H 2750 9350 50  0001 C CNN
+	1    2550 9350
+	1    0    0    -1
+$EndComp
+Wire Wire Line
+	2300 9350 2550 9350
+Connection ~ 2300 9350
+Wire Wire Line
+	2300 9350 2300 9450
+Wire Wire Line
+	2600 8200 2600 8250
+Connection ~ 2600 8250
+Wire Wire Line
+	2600 8250 3000 8250
 $EndSCHEMATC
